File: devices/pcb_solar_splitter/kicad/spliter_solar_panels.kicad_sch (KiCad schematic)
At the start: 18 parts, among them J1 Conn_01x02, J10 Conn_01x02, J2 Conn_01x02, J3 Conn_01x02, J4 Conn_01x02, J5 Conn_01x02, J6 Conn_01x02, J7 Conn_01x02, J8 Conn_01x02, J9 Conn_01x02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

Commit message: add resistances
Parts:
- added R4: 1K, symbol Device:R
- R2: value R -> 22K
- R3: value R -> 560
Connections:
- net +5V: now also U3.2 (VDD)
- net GND: now also R4.2
- net GNDREF: now also R4.1
Changed lines of the file:
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@@
   (junction (at 138.43 128.27) (diameter 0) (color 0 0 0 0)
   )
+  (junction (at 156.21 71.12) (diameter 0) (color 0 0 0 0)
+  )
   (junction (at 130.81 127) (diameter 0) (color 0 0 0 0)
   )
@@
     (stroke (width 0) (type default))
   )
+  (wire (pts (xy 158.75 71.12) (xy 156.21 71.12))
+    (stroke (width 0) (type default))
+  )
   (wire (pts (xy 132.08 105.41) (xy 132.08 104.14))
     (stroke (width 0) (type default))
@@
     (stroke (width 0) (type default))
   )
+  (wire (pts (xy 168.91 71.12) (xy 166.37 71.12))
+    (stroke (width 0) (type default))
+  )
   (wire (pts (xy 173.99 88.9) (xy 176.53 88.9))
     (stroke (width 0) (type default))
@@
   )
   (wire (pts (xy 119.38 104.14) (xy 119.38 105.41))
+    (stroke (width 0) (type default))
+  )
+  (wire (pts (xy 156.21 71.12) (xy 156.21 64.77))
     (stroke (width 0) (type default))
   )
@@
       (effects (font (size 1.27 1.27)) (justify left))
     )
-    (property "Value" "R" (at 158.75 54.61 0)
+    (property "Value" "22K" (at 158.75 54.61 0)
       (effects (font (size 1.27 1.27)) (justify left))
     )
@@
         (path "/7fb45d0e-e661-400d-950b-a242a5c78873"
           (reference "R2") (unit 1)
+        )
+      )
+    )
+  )
+  (symbol (lib_id "power:+5V") (at 74.93 52.07 0) (unit 1)
+    (in_bom yes) (on_board yes) (dnp no) (fields_autoplaced)
+    (property "Reference" "#PWR010" (at 74.93 55.88 0)
+      (effects (font (size 1.27 1.27)) hide)
+    )
+    (property "Value" "+5V" (at 74.93 46.99 0)
+      (effects (font (size 1.27 1.27)))
+    )
+    (property "Footprint" "" (at 74.93 52.07 0)
+      (effects (font (size 1.27 1.27)) hide)
+    )
+    (property "Datasheet" "" (at 74.93 52.07 0)
+      (effects (font (size 1.27 1.27)) hide)
+    )
+    (pin "1")
+    (instances
+      (project "spliter_solar_panels"
+        (path "/7fb45d0e-e661-400d-950b-a242a5c78873"
+          (reference "#PWR010") (unit 1)
         )
       )
@@
     )
   )
-  (symbol (lib_id "power:GNDREF") (at 156.21 64.77 0) (unit 1)
-    (in_bom yes) (on_board yes) (dnp no) (fields_autoplaced)
-    (property "Reference" "#PWR02" (at 156.21 71.12 0)
-      (effects (font (size 1.27 1.27)) hide)
-    )
-    (property "Value" "GNDREF" (at 156.21 69.85 0)
+  (symbol (lib_id "power:GNDREF") (at 156.21 71.12 0) (unit 1)
+    (in_bom yes) (on_board yes) (dnp no) (fields_autoplaced)
+    (property "Reference" "#PWR02" (at 156.21 77.47 0)
+      (effects (font (size 1.27 1.27)) hide)
+    )
+    (property "Value" "GNDREF" (at 156.21 76.2 0)
       (effects (font (size 1.27 1.27)))
     )
-    (property "Footprint" "" (at 156.21 64.77 0)
-      (effects (font (size 1.27 1.27)) hide)
-    )
-    (property "Datasheet" "" (at 156.21 64.77 0)
+    (property "Footprint" "" (at 156.21 71.12 0)
+      (effects (font (size 1.27 1.27)) hide)
+    )
+    (property "Datasheet" "" (at 156.21 71.12 0)
       (effects (font (size 1.27 1.27)) hide)
     )
@@
         (path "/7fb45d0e-e661-400d-950b-a242a5c78873"
           (reference "J2") (unit 1)
+        )
+      )
+    )
+  )
+  (symbol (lib_id "power:GND") (at 168.91 71.12 0) (unit 1)
+    (in_bom yes) (on_board yes) (dnp no) (fields_autoplaced)
+    (property "Reference" "#PWR011" (at 168.91 77.47 0)
+      (effects (font (size 1.27 1.27)) hide)
+    )
+    (property "Value" "GND" (at 168.91 76.2 0)
+      (effects (font (size 1.27 1.27)))
+    )
+    (property "Footprint" "" (at 168.91 71.12 0)
+      (effects (font (size 1.27 1.27)) hide)
+    )
+    (property "Datasheet" "" (at 168.91 71.12 0)
+      (effects (font (size 1.27 1.27)) hide)
+    )
+    (pin "1")
+    (instances
+      (project "spliter_solar_panels"
+        (path "/7fb45d0e-e661-400d-950b-a242a5c78873"
+          (reference "#PWR011") (unit 1)
         )
       )
@@
       (effects (font (size 1.27 1.27)) (justify left))
     )
-    (property "Value" "R" (at 158.75 62.23 0)
+    (property "Value" "560" (at 158.75 62.23 0)
       (effects (font (size 1.27 1.27)) (justify left))
     )
@@
         )
       )
+    )
+  )
+  (symbol (lib_id "Device:R") (at 162.56 71.12 90) (unit 1)
+    (in_bom yes) (on_board yes) (dnp no) (fields_autoplaced)
+    (property "Reference" "R4" (at 162.56 64.77 90)
+      (effects (font (size 1.27 1.27)))
+    )
+    (property "Value" "1K" (at 162.56 67.31 90)
+      (effects (font (size 1.27 1.27)))
+    )
+    (property "Footprint" "" (at 162.56 72.898 90)
+      (effects (font (size 1.27 1.27)) hide)
+    )
+    (property "Datasheet" "~" (at 162.56 71.12 0)
+      (effects (font (size 1.27 1.27)) hide)
+    )
+    (pin "1")
+    (pin "2")
+    (instances
+      (project "spliter_solar_panels"
+        (path "/7fb45d0e-e661-400d-950b-a242a5c78873"
+          (reference "R4") (unit 1)
+        )
+      )
